File: schema/schema_esp32/schema_esp32.kicad_sch (KiCad schematic)
At the start: 4 parts, among them U4 MAX98357A

Commit message: mic test
Connections:
- net at U2.3 (Phone_MIC_B): now also U1.34 (GPIO_34)
Changed lines of the file:
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@@
+	(wire
+		(pts
+			(xy 116.84 52.07) (xy 46.99 52.07)
+		)
+		(stroke
+			(width 0)
+			(type default)
+		)
+	)
+	(wire
+		(pts
+			(xy 43.18 82.55) (xy 46.99 82.55)
+		)
+		(stroke
+			(width 0)
+			(type default)
+		)
+	)
 	(wire
 		(pts
@@
 	(wire
 		(pts
+			(xy 116.84 76.2) (xy 116.84 52.07)
+		)
+		(stroke
+			(width 0)
+			(type default)
+		)
+	)
+	(wire
+		(pts
 			(xy 116.84 125.73) (xy 116.84 99.06)
 		)
@@
 		(pts
 			(xy 58.42 71.12) (xy 52.07 71.12)
+		)
+		(stroke
+			(width 0)
+			(type default)
+		)
+	)
+	(wire
+		(pts
+			(xy 46.99 52.07) (xy 46.99 82.55)
 		)
 		(stroke
@@
 		(pin "27"
 		)
+		(pin "34"
+		)
 		(instances
